File: merkur-22m0/merkur-22m0.brd (EAGLE design)
At the start: 35 x 23.9 mm, 7 parts, among them IC1 DERFMEGA128-XXM10

Commit message: bugfix AVDD, add pin13 PB4 PCINT4 -> configuration pin
Parts:
- SV2: device con-lsta:FE12 -> con-lsta:FE13
- moved SV2 1.27 mm to (17.8, 22.1)
Connections:
- new net N$24: IC1.24, SV2.13
- net +3V3: no longer IC1.38
Routing:
- net N$24: track 0.00 -> 14.7 mm
- net +3V3: track 69.7 -> 59.5 mm
Other:
- board text added: "1.0"
Changed lines of the file:
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@@
 <wire x1="34.976" y1="23.866" x2="0.008" y2="23.866" width="0" layer="20"/>
 <wire x1="0.008" y1="23.866" x2="0.008" y2="0" width="0" layer="20"/>
+<text x="7.62" y="16.51" size="1.27" layer="16" rot="MR0">1.0</text>
 </plain>
 <attributes>
@@
 <attribute name="OC_FARNELL" value="unknown" x="48.26" y="-14.732" size="1.778" layer="27" display="off"/>
 </element>
-<element name="SV2" library="con-lsta" package="FE12" value="" x="19.05" y="22.098" rot="R180">
-<attribute name="OC_NEWARK" value="unknown" x="-10.16" y="44.958" size="1.778" layer="27" rot="R180" display="off"/>
-<attribute name="MPN" value="" x="-10.16" y="44.958" size="1.778" layer="27" rot="R180" display="off"/>
-<attribute name="MF" value="" x="-10.16" y="44.958" size="1.778" layer="27" rot="R180" display="off"/>
-<attribute name="OC_FARNELL" value="unknown" x="-10.16" y="44.958" size="1.778" layer="27" rot="R180" display="off"/>
+<element name="SV2" library="con-lsta" package="FE13" value="" x="17.78" y="22.098" rot="R180">
+<attribute name="OC_NEWARK" value="unknown" x="-11.43" y="44.958" size="1.778" layer="27" rot="R180" display="off"/>
+<attribute name="MPN" value="" x="-11.43" y="44.958" size="1.778" layer="27" rot="R180" display="off"/>
+<attribute name="MF" value="" x="-11.43" y="44.958" size="1.778" layer="27" rot="R180" display="off"/>
+<attribute name="OC_FARNELL" value="unknown" x="-11.43" y="44.958" size="1.778" layer="27" rot="R180" display="off"/>
 </element>
 <element name="SV3" library="con-lsta" package="FE06" value="" x="1.905" y="11.303" rot="R90">
@@
 <wire x1="1.905" y1="10.033" x2="7.214" y2="10.033" width="0.4064" layer="1"/>
 <wire x1="7.214" y1="10.033" x2="7.214" y2="7.832" width="0.4064" layer="1"/>
-<contactref element="IC1" pad="38"/>
-<wire x1="18.415" y1="8.763" x2="17.145" y2="7.493" width="0.254" layer="1"/>
-<wire x1="26.67" y1="8.763" x2="18.415" y2="8.763" width="0.254" layer="1"/>
-<wire x1="17.145" y1="7.493" x2="17.05" y2="7.638" width="0.254" layer="1"/>
 <wire x1="26.67" y1="8.763" x2="26.649" y2="8.922" width="0.254" layer="1"/>
 </signal>
@@
 <via x="28.297" y="9.357" extent="1-16" drill="0.2"/>
 </signal>
+<signal name="N$24">
+<contactref element="IC1" pad="24"/>
+<contactref element="SV2" pad="13"/>
+<wire x1="11.35" y1="13.938" x2="6.35" y2="13.938" width="0.4064" layer="1"/>
+<wire x1="6.35" y1="13.938" x2="6.35" y2="13.97" width="0.4064" layer="1"/>
+<wire x1="6.35" y1="13.97" x2="3.81" y2="16.51" width="0.4064" layer="1"/>
+<wire x1="3.81" y1="16.51" x2="3.81" y2="20.32" width="0.4064" layer="1"/>
+<wire x1="3.81" y1="20.32" x2="2.54" y2="21.59" width="0.4064" layer="1"/>
+<wire x1="2.54" y1="21.59" x2="2.54" y2="22.098" width="0.4064" layer="1"/>
+</signal>
 </signals>
