File: merkur-22m0/merkur-22m0.sch (EAGLE design)
At the start: 7 parts, among them IC1 DERFMEGA128-XXM10

Commit message: bugfix AVDD, add pin13 PB4 PCINT4 -> configuration pin
Parts:
- SV2: device con-lsta:FE12-1 -> con-lsta:FE13-1
Connections:
- new net N$24: IC1.PB4/OC2A/PCINT4, SV2.13
- net +3V3: no longer IC1.AVDD
Changed lines of the file:
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@@
 <schematic xreflabel="%F%N/%S.%C%R" xrefpart="/%S.%C%R">
 <attributes>
+<attribute name="REVISION" value="1.0"/>
 </attributes>
 <variantdefs>
@@
 <part name="+3V1" library="supply1" deviceset="+3V3" device=""/>
 <part name="SV1" library="con-lsta" deviceset="FE12-1" device=""/>
-<part name="SV2" library="con-lsta" deviceset="FE12-1" device=""/>
+<part name="SV2" library="con-lsta" deviceset="FE13-1" device=""/>
 <part name="GND3" library="supply1" deviceset="GND" device=""/>
 <part name="SV3" library="con-lsta" deviceset="FE06-1" device=""/>
@@
 <part name="U$1" library="Pad" deviceset="PAD" device=""/>
 <part name="GND2" library="supply1" deviceset="GND" device=""/>
-<part name="+3V5" library="supply1" deviceset="+3V3" device=""/>
 <part name="GND5" library="supply1" deviceset="GND" device=""/>
 </parts>
@@
 <sheet>
 <plain>
+<text x="254" y="7.62" size="1.778" layer="91">&gt;REVISION</text>
 </plain>
 <instances>
@@
 <instance part="+3V1" gate="G$1" x="182.88" y="101.6"/>
 <instance part="SV1" gate="G$1" x="33.02" y="111.76"/>
-<instance part="SV2" gate="G$1" x="33.02" y="73.66" rot="MR180"/>
+<instance part="SV2" gate="G$1" x="33.02" y="71.12" rot="MR180"/>
 <instance part="GND3" gate="1" x="43.18" y="152.4"/>
 <instance part="SV3" gate="G$1" x="33.02" y="162.56"/>
@@
 <instance part="U$1" gate="G$1" x="187.96" y="68.58"/>
 <instance part="GND2" gate="1" x="101.6" y="127"/>
-<instance part="+3V5" gate="G$1" x="99.06" y="101.6"/>
 <instance part="GND5" gate="1" x="172.72" y="99.06"/>
 </instances>
@@
 <pinref part="LED2" gate="G$1" pin="A"/>
 </segment>
-<segment>
-<pinref part="+3V5" gate="G$1" pin="+3V3"/>
-<wire x1="99.06" y1="99.06" x2="99.06" y2="93.98" width="0.1524" layer="91"/>
-<pinref part="IC1" gate="G$1" pin="AVDD"/>
-<wire x1="99.06" y1="93.98" x2="101.6" y2="93.98" width="0.1524" layer="91"/>
-</segment>
 </net>
 <net name="RFOUT" class="0">
@@
 </segment>
 </net>
+<net name="N$24" class="0">
+<segment>
+<pinref part="IC1" gate="G$1" pin="PB4/OC2A/PCINT4"/>
+<wire x1="167.64" y1="147.32" x2="180.34" y2="147.32" width="0.1524" layer="91"/>
+<wire x1="180.34" y1="147.32" x2="180.34" y2="167.64" width="0.1524" layer="91"/>
+<wire x1="180.34" y1="167.64" x2="81.28" y2="167.64" width="0.1524" layer="91"/>
+<wire x1="81.28" y1="167.64" x2="81.28" y2="93.98" width="0.1524" layer="91"/>
+<wire x1="81.28" y1="93.98" x2="66.04" y2="93.98" width="0.1524" layer="91"/>
+<wire x1="66.04" y1="93.98" x2="66.04" y2="55.88" width="0.1524" layer="91"/>
+<pinref part="SV2" gate="G$1" pin="13"/>
+<wire x1="66.04" y1="55.88" x2="40.64" y2="55.88" width="0.1524" layer="91"/>
+</segment>
+</net>
